File: IR_array.kicad_sch (KiCad schematic)
At the start: 32 parts

Commit message: Finalized Scematics and Footprint
Parts:
- D1, D11, D13, D15, D3, D5, D7, D9: footprint LED_THT:LED_D3.0mm_IRBlack -> LED_THT:LED_D5.0mm
- D10, D12, D14, D16, D2, D4, D6, D8: footprint OptoDevice:Kodenshi_LG206D -> LED_THT:LED_D5.0mm_IRBlack
- R1, R10, R11, R12, R13, R14, R15, R16, R2, R3, R4, R5, R6, R7, R8, R9: value R -> 10k; footprint Package_DIP:DIP-8_W7.62mm -> Resistor_THT:R_Axial_DIN0204_L3.6mm_D1.6mm_P5.08mm_Horizontal
Connections:
- net A2: now also D6.2 (A), R6.2; no longer D4.2 (A), R4.2
- net A3: now also D10.2 (A), R10.2; no longer D6.2 (A), R6.2
- net A4: now also D14.2 (A), R14.2; no longer D8.2 (A), R8.2
- net A5: now also D4.2 (A), R4.2; no longer D10.2 (A), R10.2
- net A6: now also D8.2 (A), R8.2; no longer D12.2 (A), R12.2
- net A7: now also D12.2 (A), R12.2; no longer D14.2 (A), R14.2

Commit message: update resistor
Parts:
- R1, R11, R12, R13, R14, R15, R16, R3, R4, R5, R6, R7, R8, R9: value 10k -> 220
Changed lines of the file:
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@@
 			)
 		)
-		(property "Value" "10k"
+		(property "Value" "220"
 			(at 172.72 60.96 90)
 			(show_name no)
@@
 			)
 		)
-		(property "Value" "10k"
+		(property "Value" "220"
 			(at 172.72 86.36 90)
 			(show_name no)
@@
 			)
 		)
-		(property "Value" "10k"
+		(property "Value" "220"
 			(at 172.72 46.99 90)
 			(show_name no)
@@
 			)
 		)
-		(property "Value" "10k"
+		(property "Value" "220"
 			(at 86.36 45.72 90)
 			(show_name no)
@@
 			)
 		)
-		(property "Value" "10k"
+		(property "Value" "220"
 			(at 46.99 45.72 90)
 			(show_name no)
@@
 			)
 		)
-		(property "Value" "10k"
+		(property "Value" "220"
 			(at 86.36 59.69 90)
 			(show_name no)
@@
 			)
 		)
-		(property "Value" "10k"
+		(property "Value" "220"
 			(at 86.36 85.09 90)
 			(show_name no)
@@
 			)
 		)
-		(property "Value" "10k"
+		(property "Value" "220"
 			(at 125.73 99.06 90)
 			(show_name no)
@@
 			)
 		)
-		(property "Value" "10k"
+		(property "Value" "220"
 			(at 125.73 45.72 90)
 			(show_name no)
@@
 			)
 		)
-		(property "Value" "10k"
+		(property "Value" "220"
 			(at 46.99 99.06 90)
 			(show_name no)
@@
 			)
 		)
-		(property "Value" "10k"
+		(property "Value" "220"
 			(at 46.99 85.09 90)
 			(show_name no)
@@
 			)
 		)
-		(property "Value" "10k"
+		(property "Value" "220"
 			(at 86.36 99.06 90)
 			(show_name no)
@@
 			)
 		)
-		(property "Value" "10k"
+		(property "Value" "220"
 			(at 125.73 85.09 90)
 			(show_name no)
@@
 			)
 		)
-		(property "Value" "10k"
+		(property "Value" "220"
 			(at 172.72 100.33 90)
 			(show_name no)
