File: VacumBlocks.kicad_pcb (KiCad board)
At the start: 2 copper layers, 42 parts, among them J1 Conn_01x03_Socket, J2 Screw_Terminal_01x04, J3 Conn_01x03_Socket, J4 Conn_01x03_Socket, M5 TB6612FNG_module, U2 Nodemcu-32S

Commit message: Adding of the screw terminal block and schematics PDF
Parts:
- added J5: Screw_Terminal_01x03, TerminalBlock:TerminalBlock_MaiXu_MX126-5.0-03P_1x03_P5.00mm, F.Cu at (30.2, 98.0)
- R1, R11, R12, R13, R14, R15, R16, R3, R4, R5, R6, R7, R8, R9: value 10k -> 220
